File: bootmode/arduino/Hardware/h8_ztat_flasher.kicad_sch (KiCad schematic)
At the start: 11 parts, among them J1 Conn_02x05_Counter_Clockwise, Q1 B1187? ~1A or so peak, Q2 NPN?, Q3 PNP? ~300mA or so?

Commit message: cleanup: ztat_flasher: bin stray resistor
Parts:
- removed R6: 10k0, symbol Device:R
Changed lines of the file:
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@@
   (junction (at 176.53 91.44) (diameter 0) (color 0 0 0 0)
-  )
-  (junction (at 176.53 93.98) (diameter 0) (color 0 0 0 0)
   )
   (junction (at 165.1 86.36) (diameter 0) (color 0 0 0 0)
@@
     (stroke (width 0) (type default))
   )
-  (wire (pts (xy 176.53 93.98) (xy 176.53 96.52))
-    (stroke (width 0) (type default))
-  )
   (wire (pts (xy 154.94 109.22) (xy 157.48 109.22))
     (stroke (width 0) (type default))
@@
   (label "PRG_TX" (at 106.68 99.06 0) (fields_autoplaced)
     (effects (font (size 1.27 1.27)) (justify left bottom))
-  )
-  (symbol (lib_id "Device:R") (at 180.34 96.52 90) (unit 1)
-    (in_bom yes) (on_board yes) (dnp no)
-    (property "Reference" "R6" (at 180.34 99.06 90)
-      (effects (font (size 1.27 1.27)))
-    )
-    (property "Value" "10k0" (at 180.34 96.52 90)
-      (effects (font (size 1.27 1.27)))
-    )
-    (property "Footprint" "" (at 180.34 98.298 90)
-      (effects (font (size 1.27 1.27)) hide)
-    )
-    (property "Datasheet" "~" (at 180.34 96.52 0)
-      (effects (font (size 1.27 1.27)) hide)
-    )
-    (pin "1")
-    (pin "2")
-    (instances
-      (project "flasher"
-        (path "/27b5d8bd-cefd-4a1e-8ed3-661b96ace440"
-          (reference "R6") (unit 1)
-        )
-      )
-    )
   )
   (symbol (lib_id "Connector_Generic:Conn_02x05_Counter_Clockwise") (at 85.09 101.6 0) (unit 1)
@@
     (pin "8")
     (instances
-      (project "flasher"
+      (project "h8_ztat_flasher"
         (path "/27b5d8bd-cefd-4a1e-8ed3-661b96ace440"
           (reference "J1") (unit 1)
@@
     (pin "1")
     (instances
-      (project "flasher"
+      (project "h8_ztat_flasher"
         (path "/27b5d8bd-cefd-4a1e-8ed3-661b96ace440"
           (reference "#PWR03") (unit 1)
@@
     (pin "3")
     (instances
-      (project "flasher"
+      (project "h8_ztat_flasher"
         (path "/27b5d8bd-cefd-4a1e-8ed3-661b96ace440"
           (reference "Q3") (unit 1)
@@
     (pin "20")
     (instances
-      (project "flasher"
+      (project "h8_ztat_flasher"
         (path "/27b5d8bd-cefd-4a1e-8ed3-661b96ace440"
           (reference "A1") (unit 1)
@@
     (pin "2")
     (instances
-      (project "flasher"
+      (project "h8_ztat_flasher"
         (path "/27b5d8bd-cefd-4a1e-8ed3-661b96ace440"
           (reference "R5") (unit 1)
@@
     (pin "1")
     (instances
-      (project "flasher"
+      (project "h8_ztat_flasher"
         (path "/27b5d8bd-cefd-4a1e-8ed3-661b96ace440"
           (reference "#PWR02") (unit 1)
@@
     (pin "1")
     (instances
-      (project "flasher"
+      (project "h8_ztat_flasher"
         (path "/27b5d8bd-cefd-4a1e-8ed3-661b96ace440"
           (reference "#PWR01") (unit 1)
@@
     (pin "1")
     (instances
-      (project "flasher"
+      (project "h8_ztat_flasher"
         (path "/27b5d8bd-cefd-4a1e-8ed3-661b96ace440"
           (reference "R2") (unit 1)
@@
     (pin "2")
     (instances
-      (project "flasher"
+      (project "h8_ztat_flasher"
         (path "/27b5d8bd-cefd-4a1e-8ed3-661b96ace440"
           (reference "R1") (unit 1)
@@
     (pin "3")
     (instances
-      (project "flasher"
+      (project "h8_ztat_flasher"
         (path "/27b5d8bd-cefd-4a1e-8ed3-661b96ace440"
           (reference "Q1") (unit 1)
@@
     (pin "1")
     (instances
-      (project "flasher"
+      (project "h8_ztat_flasher"
         (path "/27b5d8bd-cefd-4a1e-8ed3-661b96ace440"
           (reference "R3") (unit 1)
@@
     (pin "2")
     (instances
-      (project "flasher"
+      (project "h8_ztat_flasher"
         (path "/27b5d8bd-cefd-4a1e-8ed3-661b96ace440"
           (reference "R4") (unit 1)
@@
     (pin "2")
     (instances
-      (project "flasher"
+      (project "h8_ztat_flasher"
         (path "/27b5d8bd-cefd-4a1e-8ed3-661b96ace440"
           (reference "Q2") (unit 1)
